Commit message: Added imu sensor

File: ros_foxy_ws/install/share/two_wheel_sim/urdf/two_wheel.xacro.urdf (robot description, URDF)
Before this commit: robot Two_Wheel, 3 links, 2 joints
Links:
- added link imu_link, mass 0.001; collision box size=.001 .001 .001; visual box size=0.001 0.001 0.001
Joints:
- added joint imu_joint: type fixed, parent root, child imu_link, origin xyz=0 0 0, axis 1 0 0
