Commit message: Controller imp and testing

File: ros_foxy_ws/src/two_wheel_sim/urdf/two_wheel.xacro.urdf (robot description, URDF)
Before this commit: robot Two_Wheel, 4 links, 3 joints
Links:
- added link body, mass ${m_b}; collision box size=${l_b} ${w_b} ${h_b}; visual box size=${l_b} ${w_b} ${h_b}
- link root: mass ${m_b} -> None; geometry 
Joints:
- added joint body_joint: type fixed, parent root, child body, origin xyz=0 0 0 rpy=0 0 0
- joint LW_joint: axis (none) -> 1 0 0; limit effort=${eff_lim} velocity=${speed_lim} -> lower=-${eff_lim} upper=${eff_lim} effort=${eff_lim} velocity=${speed_lim}; parent root -> body
- joint RW_joint: axis (none) -> 1 0 0; limit effort=${eff_lim} velocity=${speed_lim} -> lower=-${eff_lim} upper=${eff_lim} effort=${eff_lim} velocity=${speed_lim}; parent root -> body
- joint imu_joint: parent root -> body

Commit message: Added filtering on theta y and tuned PID

File: ros_foxy_ws/src/two_wheel_sim/urdf/two_wheel.xacro.urdf (robot description, URDF)
Before this commit: robot Two_Wheel, 5 links, 4 joints
Links:
- removed link body
- added link base_link, mass ${m_b}; collision box size=${l_b} ${w_b} ${h_b}; visual box size=${l_b} ${w_b} ${h_b}
Joints:
- removed joint body_joint
- added joint base_link_joint: type fixed, parent root, child base_link, origin xyz=0 0 0 rpy=0 0 0
- joint LW_joint: parent body -> base_link
- joint RW_joint: parent body -> base_link
- joint imu_joint: parent body -> base_link

Commit message: Adapted urdf and controller to convention (x forward)

File: ros_foxy_ws/src/two_wheel_sim/urdf/two_wheel.xacro.urdf (robot description, URDF)
Before this commit: robot Two_Wheel, 5 links, 4 joints
Joints:
- joint LW_joint: axis 1 0 0 -> 0 1 0; origin xyz=${-l_b/2} 0 ${-h_b/2} rpy=0.0 0.0 0.0 -> xyz=0 ${-w_b/2} ${-h_b/2} rpy=0.0 0.0 0.0
- joint RW_joint: axis 1 0 0 -> 0 1 0; origin xyz=${l_b/2} 0 ${-h_b/2} rpy=0.0 0.0 0.0 -> xyz=0 ${w_b/2} ${-h_b/2} rpy=0.0 0.0 0.0

Commit message: Added Odometry and ekf position estimation

File: ros_foxy_ws/src/two_wheel_sim/urdf/two_wheel.xacro.urdf (robot description, URDF)
Before this commit: robot Two_Wheel, 5 links, 4 joints
Links:
- removed link root
- added link body, mass ${m_b}; collision box size=${l_b} ${w_b} ${h_b}; visual box size=${l_b} ${w_b} ${h_b}
- link base_link: mass ${m_b} -> None; geometry 
Joints:
- removed joint base_link_joint
- added joint body_joint: type fixed, parent base_link, child body, origin xyz=0 0 ${h_b/2} rpy=0 0 0
- joint LW_joint: parent base_link -> body
- joint RW_joint: parent base_link -> body
- joint imu_joint: parent base_link -> body

Commit message: started working on navigation

File: ros_foxy_ws/src/two_wheel_sim/urdf/two_wheel.xacro.urdf (robot description, URDF)
Before this commit: robot Two_Wheel, 5 links, 4 joints
Links:
- added link base_footprint
- added link lidar_link, mass 0.001; collision box size=.001 .001 .001; visual box size=0.001 0.001 0.001
Joints:
- added joint footprint_joint: type fixed, parent base_link, child base_footprint, origin xyz=0 0 ${-r_w * 0.5} rpy=0 0 0
- added joint lidar_joint: type fixed, parent body, child lidar_link, origin xyz=${l_b/2 + 0.1} 0 0, axis 1 0 0
